File: hw/Dash Motor.kicad_sch (KiCad schematic)
At the start: 73 parts, among them CN1 SM07B-SRSS-TB(LF)(SN), CN2 XT30PW-M30.G.Y, CN3 XY119A-5.0-3P, U2 DRV8323RSRGZT, U4 MA732GQ-Z, U5 MCP2542FD-E/MF, U6 S3B-PH-SM4-TB(LF)(SN), U7 AMS1117-3.3, X2 8MHz

Commit message: Add files via upload
Parts:
- removed CN2: XT30PW-M30.G.Y, Dash Motor-easyedapro:CONN-TH_XT30PW-M, symbol Dash Motor-easyedapro:XT30PW-M
- added CN2(IN), CN3(OUT): XT30(2+2)PB-M.G.B, Footprints:CONN-TH_XT30PB-M, symbol Changzhou Amass Elec XT30(2+2)PB-M.G.B:XT30(2+2)PB-M.G.B
Connections:
- net 3V3: now also CN2(IN).2 (3.3V+), CN3(OUT).2 (3.3V+)
- net GND: now also CN2(IN).1 (3.3V-), CN2(IN).3 (48V-), CN3(OUT).1 (3.3V-), CN3(OUT).3 (48V-)
- net 24V renamed 48V
- net 48V: now also CN2(IN).4 (48V+), CN3(OUT).4 (48V+)
Other:
- moved on the sheet: C1, C11, C12, C13, C14, C15, C16, C21, C22, C23, C24, C25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
